File: PCBs/EC-DLM-TR05/kicadProject/ec-dlm-tr04.sch (KiCad schematic (older format))
At the start: 23 parts, among them J1 input, J2 LED Connector, J3 RJ45, U1 MCP6424, U2 LD1117S50TR

Commit message: no message
Parts:
- added C?: 105, Capacitors_THT:CP_Radial_D4.0mm_P2.00mm, symbol C
- added R?: 10k, Resistors_THT:R_Axial_DIN0207_L6.3mm_D2.5mm_P7.62mm_Horizontal, symbol R
- C1: value 104 -> 105
Connections:
- net ADCInput: now also C?.1, R?.2; no longer R6.2, R8.1, U1.8
- net GND: now also C?.2
- new net: R6.2, R8.1, R?.1, U1.8
Changed lines of the file:
@@
 P 6375 2700
 F 0 "C1" H 6400 2800 50  0000 L CNN
-F 1 "104" H 6400 2600 50  0000 L CNN
+F 1 "105" H 6400 2600 50  0000 L CNN
 F 2 "Capacitors_THT:CP_Radial_D4.0mm_P2.00mm" H 6413 2550 50  0001 C CNN
 F 3 "" H 6375 2700 50  0001 C CNN
@@
 Text GLabel 8925 2075 2    60   Output ~ 0
 ADCInput
-Wire Wire Line
-	5600 2075 8925 2075
 $Comp
 L D_Zener_ALT D2
@@
 Wire Wire Line
 	8250 2100 8250 2075
-Connection ~ 8250 2075
 Wire Wire Line
 	6725 2525 7050 2525
@@
 Wire Wire Line
 	1350 5550 1350 5500
+$Comp
+L R R?
+U 1 1 5C44BBA8
+P 6000 2075
+F 0 "R?" V 6080 2075 50  0000 C CNN
+F 1 "10k" V 6000 2075 50  0000 C CNN
+F 2 "Resistors_THT:R_Axial_DIN0207_L6.3mm_D2.5mm_P7.62mm_Horizontal" V 5930 2075 50  0001 C CNN
+F 3 "" H 6000 2075 50  0001 C CNN
+	1    6000 2075
+	0    -1   -1   0
+$EndComp
+Wire Wire Line
+	5850 2075 5600 2075
+$Comp
+L C C?
+U 1 1 5C44BCEB
+P 6375 1925
+F 0 "C?" H 6400 2025 50  0000 L CNN
+F 1 "105" H 6400 1825 50  0000 L CNN
+F 2 "Capacitors_THT:CP_Radial_D4.0mm_P2.00mm" H 6413 1775 50  0001 C CNN
+F 3 "" H 6375 1925 50  0001 C CNN
+	1    6375 1925
+	-1   0    0    1
+$EndComp
+Wire Wire Line
+	6150 2075 8925 2075
+Connection ~ 6375 2075
+Wire Wire Line
+	8250 2075 8350 2075
+Connection ~ 8350 2075
+Connection ~ 8250 2075
+$Comp
+L GND #PWR?
+U 1 1 5C44BFD3
+P 6150 1750
+F 0 "#PWR?" H 6150 1500 50  0001 C CNN
+F 1 "GND" H 6150 1600 50  0000 C CNN
+F 2 "" H 6150 1750 50  0001 C CNN
+F 3 "" H 6150 1750 50  0001 C CNN
+	1    6150 1750
+	1    0    0    -1
+$EndComp
+Wire Wire Line
+	6150 1750 6150 1700
+Wire Wire Line
+	6150 1700 6375 1700
+Wire Wire Line
+	6375 1700 6375 1775
 $EndSCHEMATC

Commit message: TR04 + DLM01 REV9 adjustments.
Parts:
- removed C1: 105, Capacitors_THT:CP_Radial_D4.0mm_P2.00mm, symbol C
- removed D3: BZX79C3V3‎, Diodes_THT:D_DO-35_SOD27_P7.62mm_Horizontal, symbol D_Zener_ALT
- removed R10: 33k, Resistors_THT:R_Axial_DIN0207_L6.3mm_D2.5mm_P7.62mm_Horizontal, symbol R
- removed R11, R9: 470k, Resistors_THT:R_Axial_DIN0207_L6.3mm_D2.5mm_P7.62mm_Horizontal, symbol R
- removed R3, R8: 10k, Resistors_THT:R_Axial_DIN0207_L6.3mm_D2.5mm_P7.62mm_Horizontal, symbol R
- R2: value 7.5k -> 10k
- gave numbers to parts that had none: 2
Connections:
- net RESET is gone; now on net GND: J3.2
- net +5V: now also J3.8; no longer C2.1, C3.1, J3.5, U1.4 (V+), U1.4 (V+), U1.4 (V+), U1.4 (V+)
- net GND: no longer C1.2, C2.2, C3.2, D2.2 (A), J1.1 (P1), J3.3, U1.11 (V-), U1.11 (V-), U1.11 (V-), U1.11 (V-), U1.5 (+)
- net at R4.2, U1.7: now also U1.5 (+)
- net AGND: now reaches U1.12 (+)
- net AGND: now also C1.1, C2.2, C3.2, D2.2 (A), J1.1 (P1), J3.3, U1.11 (V-), U1.11 (V-), U1.11 (V-), U1.11 (V-)
- net at U1.13 (-): now also U1.14
- net ADCInput renamed ADCTrig
- net ADCTrig: now also C1.2; no longer C1.1
- net SchmidtTrigInput renamed AVCC
- net AVCC: now also C2.1, C3.1, U1.4 (V+), U1.4 (V+), U1.4 (V+), U1.4 (V+); no longer U1.14
- net WSLED-Signal renamed L_OUT_5
- net L_OUT_5: now also J3.5; no longer J3.8
- no-connect marks 2 -> 1
Other:
- note added: "LED Strip connection"
- note added: "Low pass filter at 4.8kHz"
- note added: "Main Module interface"
- note added: "Unused opamp channel"
- note added: "Voltage regulator for LEDS \n(optionnal, bypass by shorting 3 and 2 pins with a jumper)"
- note removed: "3.3v clipping\ndiodes"
- note removed: "Low pass filter \nat 4.8kHz"
- note removed: "Pot for control \nof trigger sensitivity"
- note removed: "Schmidt trigger\ncircuit\n(with hysteresis resistor)"
- moved on the sheet: C1, C2, C3, D2, J2, J3, R2, U1D

Commit message: New Main board.
Parts:
- removed C4: 105, Capacitors_THT:CP_Radial_D4.0mm_P2.00mm, symbol C
- removed C5: 4.7pF, Capacitors_THT:CP_Radial_D4.0mm_P2.00mm, symbol C
- removed U2: LD1117S50TR, TO_SOT_Packages_SMD:SOT-223, symbol LD1117S50TR
- added C? (x2): 10u, symbol CP
- added C?: 100u, symbol CP
- added U?: TC1044S, symbol TC1044S
- U1: value MCP6424 -> TL074
Connections:
- net AGND: now also C?.1, U?.3 (GND); no longer U1.11 (V-), U1.11 (V-), U1.11 (V-), U1.11 (V-)
- net AVCC: now also C?.1, U?.1 (Boost), U?.8 (V+)
- net at R1.1, U1.6 (-): now also U1.5 (+); no longer U1.3 (+)
- new net: R2.2, U1.6 (-), U1.7
- new net: C?.1, U?.2 (Cap+)
- new net: C?.2, U?.4 (cap-)
- new net AVSS: C?.2, C?.2, U1.11 (V-), U1.11 (V-), U1.11 (V-), U1.11 (V-), U?.5 (vOut)
- no-connect marks 1 -> 3
Other:
- note added: "Negative supply for opamp"
- note removed: "Voltage regulator for LEDS \n(optionnal, bypass by shorting 3 and 2 pins with a jumper)"
Changed lines of the file:
@@
 $Comp
 L TL084 U1
-U 1 1 5BEAA9C2
+U 2 1 5BEAA9C2
 P 2500 2475
 F 0 "U1" H 2500 2675 50  0000 L CNN
-F 1 "MCP6424" H 2500 2275 50  0000 L CNN
+F 1 "TL074" H 2500 2275 50  0000 L CNN
 F 2 "SMD_Packages:SOIC-14_N" H 2450 2575 50  0001 C CNN
 F 3 "" H 2550 2675 50  0001 C CNN
-	1    2500 2475
+	2    2500 2475
 	1    0    0    -1
 $EndComp
@@
 P 5250 2475
 F 0 "U1" H 5250 2675 50  0000 L CNN
-F 1 "MCP6424" H 5225 2300 50  0000 L CNN
+F 1 "TL074" H 5225 2300 50  0000 L CNN
 F 2 "SMD_Packages:SOIC-14_N" H 5200 2575 50  0001 C CNN
 F 3 "" H 5300 2675 50  0001 C CNN
@@
 P 4025 2375
 F 0 "U1" H 4025 2575 50  0000 L CNN
-F 1 "MCP6424" H 3975 2200 50  0000 L CNN
+F 1 "TL074" H 3975 2200 50  0000 L CNN
 F 2 "SMD_Packages:SOIC-14_N" H 3975 2475 50  0001 C CNN
 F 3 "" H 4075 2575 50  0001 C CNN
@@
 P 8475 2375
 F 0 "U1" H 8475 2575 50  0000 L CNN
-F 1 "MCP6424" H 8475 2175 50  0000 L CNN
+F 1 "TL074" H 8475 2175 50  0000 L CNN
 F 2 "SMD_Packages:SOIC-14_N" H 8425 2475 50  0001 C CNN
 F 3 "" H 8525 2575 50  0001 C CNN
@@
 	9575 4025 9575 4950
 $Comp
-L LD1117S50TR U2
-U 1 1 5C149F08
-P 1825 5150
-F 0 "U2" H 1800 5425 50  0000 C CNN
-F 1 "LD1117S50TR" H 1825 5350 50  0000 C CNN
-F 2 "TO_SOT_Packages_SMD:SOT-223" H 1825 5250 50  0001 C CNN
-F 3 "" H 1825 5150 50  0001 C CNN
-	1    1825 5150
-	1    0    0    -1
-$EndComp
-Text GLabel 2425 5100 2    60   Input ~ 0
-VCC5-LDO
-Wire Wire Line
-	2225 5100 2425 5100
-$Comp
-L GND #PWR2
-U 1 1 5C14A3EB
-P 1825 5600
-F 0 "#PWR2" H 1825 5350 50  0001 C CNN
-F 1 "GND" H 1825 5450 50  0000 C CNN
-F 2 "" H 1825 5600 50  0001 C CNN
-F 3 "" H 1825 5600 50  0001 C CNN
-	1    1825 5600
-	1    0    0    -1
-$EndComp
-Wire Wire Line
-	1825 5400 1825 5600
-$Comp
-L C C5
-U 1 1 5C14A58F
-P 2325 5350
-F 0 "C5" H 2350 5450 50  0000 L CNN
-F 1 "4.7pF" H 2350 5250 50  0000 L CNN
-F 2 "Capacitors_THT:CP_Radial_D4.0mm_P2.00mm" H 2363 5200 50  0001 C CNN
-F 3 "" H 2325 5350 50  0001 C CNN
-	1    2325 5350
-	-1   0    0    1
-$EndComp
-$Comp
-L C C4
-U 1 1 5C14A7DC
-P 1350 5350
-F 0 "C4" H 1375 5450 50  0000 L CNN
-F 1 "105" H 1375 5250 50  0000 L CNN
-F 2 "Capacitors_THT:CP_Radial_D4.0mm_P2.00mm" H 1388 5200 50  0001 C CNN
-F 3 "" H 1350 5350 50  0001 C CNN
-	1    1350 5350
-	-1   0    0    1
-$EndComp
-Text GLabel 1175 5100 0    60   Input ~ 0
-VCC5
-Wire Wire Line
-	1175 5100 1425 5100
-Wire Wire Line
-	1350 5200 1350 5100
-Connection ~ 1350 5100
-Wire Wire Line
-	2325 5200 2325 5100
-Connection ~ 2325 5100
-Wire Wire Line
-	2325 5550 2325 5500
-Wire Wire Line
-	1350 5550 2325 5550
-Connection ~ 1825 5550
-Wire Wire Line
-	1350 5550 1350 5500
-$Comp
 L R R3
 U 1 1 5C44BBA8
@@
 Wire Wire Line
 	7175 5275 7175 5325
-Text Notes 825  4725 0    79   ~ 16
-Voltage regulator for LEDS \n(optionnal, bypass by shorting 3 and 2 pins with a jumper)
 Text GLabel 2475 2850 2    60   Output ~ 0
-AGND
+AVSS
 Wire Wire Line
 	2400 2775 2400 2850
@@
 	2400 2850 2475 2850
 Text GLabel 4000 2750 2    60   Output ~ 0
-AGND
+AVSS
 Text GLabel 5200 2850 2    60   Output ~ 0
-AGND
+AVSS
 Wire Wire Line
 	5200 2850 5150 2850
@@
 AVCC
 Text GLabel 8375 2675 2    60   Output ~ 0
-AGND
+AVSS
 Text GLabel 8175 2275 0    60   Output ~ 0
 AGND
@@
 Text Notes 7875 1900 0    79   ~ 16
 Unused opamp channel
+$Comp
+L TC1044S U?
+U 1 1 5C6DD326
+P 2475 5675
+F 0 "U?" H 2275 6025 60  0000 C CNN
+F 1 "TC1044S" H 2475 5275 60  0000 C CNN
+F 2 "" H 2475 5675 60  0001 C CNN
+F 3 "" H 2475 5675 60  0001 C CNN
+	1    2475 5675
+	1    0    0    -1
+$EndComp
+Text GLabel 3600 5475 2    60   Input ~ 0
+AVCC
+Wire Wire Line
+	1975 5475 1875 5475
+Wire Wire Line
+	1875 5475 1875 5050
+Wire Wire Line
+	1875 5050 3200 5050
+Wire Wire Line
+	3200 5050 3200 5475
+Wire Wire Line
+	3125 5475 3600 5475
+Connection ~ 3200 5475
+NoConn ~ 3125 5775
+Text GLabel 1775 5775 0    60   Output ~ 0
+AGND
+Wire Wire Line
+	1775 5775 1975 5775
+Text GLabel 3550 5925 2    60   Output ~ 0
+AVSS
+NoConn ~ 3125 5625
+$Comp
+L CP C?
+U 1 1 5C6DDAED
+P 1225 5800
+F 0 "C?" H 1250 5900 50  0000 L CNN
+F 1 "10u" H 1250 5700 50  0000 L CNN
+F 2 "" H 1263 5650 50  0001 C CNN
+F 3 "" H 1225 5800 50  0001 C CNN
+	1    1225 5800
+	1    0    0    -1
+$EndComp
+Wire Wire Line
+	1975 5625 1225 5625
+Wire Wire Line
+	1225 5625 1225 5650
+Wire Wire Line
+	1225 5950 1975 5950
+Wire Wire Line
+	1975 5950 1975 5925
+Wire Wire Line
+	3125 5925 3550 5925
+Text GLabel 3325 6375 3    60   Output ~ 0
+AGND
+$Comp
+L CP C?
+U 1 1 5C6DDDFD
+P 3325 6125
+F 0 "C?" H 3350 6225 50  0000 L CNN
+F 1 "10u" H 3350 6025 50  0000 L CNN
+F 2 "" H 3363 5975 50  0001 C CNN
+F 3 "" H 3325 6125 50  0001 C CNN
+	1    3325 6125
+	-1   0    0    1
+$EndComp
+Wire Wire Line
+	3325 6275 3325 6375
+Wire Wire Line
+	3325 5975 3325 5925
+Connection ~ 3325 5925
+Text Notes 1725 4925 0    79   ~ 16
+Negative supply for opamp
+$Comp
+L CP C?
+U 1 1 5C6DEA9E
+P 3450 5700
+F 0 "C?" H 3475 5800 50  0000 L CNN
+F 1 "100u" H 3475 5600 50  0000 L CNN
+F 2 "" H 3488 5550 50  0001 C CNN
+F 3 "" H 3450 5700 50  0001 C CNN
+	1    3450 5700
+	1    0    0    -1
+$EndComp
+Wire Wire Line
+	3450 5550 3450 5475
+Connection ~ 3450 5475
+Wire Wire Line
+	3450 5850 3450 5925
+Connection ~ 3450 5925
 $EndSCHEMATC

Commit message: Revision board rev9
Parts:
- added C7: 104, Capacitors_THT:CP_Radial_D6.3mm_P2.50mm, symbol C
- added D3, D4: D, Diodes_THT:D_A-405_P2.54mm_Vertical_AnodeUp, symbol D
- added L1: Ferrite_Bead, Inductors_THT:L_Axial_L6.6mm_D2.7mm_P2.54mm_Vertical_Vishay_IM-2, symbol Ferrite_Bead
- added R10, R7, R8, R9: 10k, Resistors_THT:R_Axial_DIN0204_L3.6mm_D1.6mm_P1.90mm_Vertical, symbol R
- C4, C5, C6: renamed from C?; footprint (none) -> Capacitors_THT:CP_Radial_D6.3mm_P2.50mm
- D2: value BZX79C3V3 -> BZX79C5V; footprint Diodes_THT:D_DO-35_SOD27_P7.62mm_Horizontal -> Diodes_THT:D_DO-35_SOD27_P2.54mm_Vertical_AnodeUp
- R1: value 27k -> 100k; footprint Resistors_THT:R_Axial_DIN0207_L6.3mm_D2.5mm_P7.62mm_Horizontal -> Resistors_THT:R_Axial_DIN0204_L3.6mm_D1.6mm_P1.90mm_Vertical
- R2, R3, R4, R5, R6: footprint Resistors_THT:R_Axial_DIN0207_L6.3mm_D2.5mm_P7.62mm_Horizontal -> Resistors_THT:R_Axial_DIN0204_L3.6mm_D1.6mm_P1.90mm_Vertical
- U2: renamed from U?; footprint (none) -> Housings_SOIC:SOIC-8_3.9x4.9mm_Pitch1.27mm
Connections:
- net VCC5-LDO is gone; now on net +5V: J2.3 (P3)
- net AGND: now also R5.2, U1.10 (+), C7.2; no longer U1.12 (+)
- net AVCC: now also L1.1; no longer C6.1, U2.1 (Boost), U2.8 (V+)
- net GND: no longer R5.1
- net at U1.6 (-), U1.7: now also D4.2 (A); no longer R2.2
- net at R3.1, R6.2: now also U1.14; no longer U1.8
- new net: R9.2, U1.5 (+)
- new net: D3.2 (A), R8.1, U1.8
- new net: R2.1, R8.2, U1.9 (-)
- new net: R10.1, U1.12 (+)
- new net: D1.1 (K), R5.1, U1.13 (-)
- new net: R4.2, R7.1, U1.1
- new net: R7.2, U1.2 (-)
- new net: R1.1, U1.3 (+)
- new net: C7.1, R2.2, R4.1, R9.1
- new net: C6.1, L1.2, U2.1 (Boost), U2.8 (V+)
- new net: D3.1 (K), D4.1 (K), R10.2
Other:
- note added: "Negative supply for opamp (+12v to -12v)"
- note removed: "Negative supply for opamp"
- note removed: "Unused opamp channel"
- moved on the sheet: C1, C2, C3, C4, C5, C6, D1, D2, J1, J2, J3, R1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

Commit message: PCB Rouge
Parts:
- removed C2: 10uf tantale, Capacitors_THT:CP_Radial_D5.0mm_P2.00mm, symbol CP1
- removed C3: 100nf cer, Capacitors_THT:CP_Radial_D5.0mm_P2.00mm, symbol CP1
- added C10: 10uf, Capacitors_THT:CP_Radial_D6.3mm_P2.50mm, symbol CP1
- added C11, C12, C3, C9: 100n, Capacitors_SMD:C_0805_HandSoldering, symbol C
- added C2: 1n, Capacitors_SMD:C_0805_HandSoldering, symbol C
- added C8: 10u, Capacitors_THT:CP_Radial_D6.3mm_P2.50mm, symbol CP1
- added R11: 10k, Resistors_SMD:R_0805_HandSoldering, symbol R
- C1: value 105 -> 100n; footprint Capacitors_THT:CP_Radial_D4.0mm_P2.00mm -> Capacitors_SMD:C_0805_HandSoldering
- C4, C5, C6: footprint Capacitors_THT:CP_Radial_D6.3mm_P2.50mm -> Capacitors_THT:CP_Radial_D4.0mm_P2.00mm
- C7: value 104 -> 10n; footprint Capacitors_THT:CP_Radial_D6.3mm_P2.50mm -> Capacitors_SMD:C_0805_HandSoldering
- D1: footprint Diodes_THT:D_DO-35_SOD27_P2.54mm_Vertical_AnodeUp -> Diodes_SMD:D_SOD-123
- D3, D4: footprint Diodes_THT:D_A-405_P2.54mm_Vertical_AnodeUp -> Diodes_SMD:D_SOD-123
- R1, R10, R2, R3, R4, R5, R6, R8, R9: footprint Resistors_THT:R_Axial_DIN0204_L3.6mm_D1.6mm_P1.90mm_Vertical -> Resistors_SMD:R_0805_HandSoldering
- R7: value 10k -> 100k; footprint Resistors_THT:R_Axial_DIN0204_L3.6mm_D1.6mm_P1.90mm_Vertical -> Resistors_SMD:R_0805_HandSoldering
Connections:
- net +5V: now also C10.1
- net AGND: now also C11.2, C12.2, C2.2, C3.2, C8.2, C9.1, R11.1
- net AVCC: now also C11.1, C8.1, C9.2
- net AVSS: now also C12.1, C3.1
- net GND: now also C10.2
- net at D4.2 (A), U1.7: no longer U1.6 (-)
- net at D3.2 (A), U1.8: no longer R8.1
- net at D1.1 (K), R5.1, U1.13 (-): now also R7.2
- net at R4.2, U1.1: now also U1.2 (-); no longer R7.1
- net at R1.1, U1.3 (+): now also C2.1
- net at D1.2 (A), R6.1: now also R7.1
- net at D3.1 (K), D4.1 (K), R10.2: now also R8.1, U1.6 (-), R11.2
Other:
- moved on the sheet: L1, R10

Commit message: Revision TR05 (Board rouge satellite) selon les tests.
Parts:
- D2: value BZX79C5V -> 1N4148
- R12: renamed from C2; value 1n -> 1M; footprint Capacitors_SMD:C_0805_HandSoldering -> Resistors_SMD:R_0805_HandSoldering; symbol C -> R
- R13: renamed from C7; value 10n -> 1M; footprint Capacitors_SMD:C_0805_HandSoldering -> Resistors_SMD:R_0805_HandSoldering; symbol C -> R
Changed lines of the file:
@@
 U 1 1 5C010B25
 P 7700 1650
-F 0 "R6" V 7850 1650 50  0000 C CNN
-F 1 "10k" V 7775 1650 50  0000 C CNN
+F 0 "R6" V 7800 1575 50  0000 C CNN
+F 1 "10k" V 7600 1550 50  0000 C CNN
 F 2 "Resistors_SMD:R_0805_HandSoldering" V 7630 1650 50  0001 C CNN
 F 3 "" H 7700 1650 50  0001 C CNN
@@
 U 1 1 5C010F9E
 P 7350 1650
-F 0 "D1" H 7350 1750 50  0000 C CNN
-F 1 "1N4148" H 7375 1550 50  0000 C CNN
+F 0 "D1" H 7250 1600 50  0000 C CNN
+F 1 "1N4148" H 7450 1550 50  0000 C CNN
 F 2 "Diodes_SMD:D_SOD-123" H 7350 1650 50  0001 C CNN
 F 3 "" H 7350 1650 50  0001 C CNN
@@
 P 8975 2225
 F 0 "D2" V 9000 2350 50  0000 C CNN
-F 1 "BZX79C5V" V 8925 2500 50  0000 C CNN
+F 1 "1N4148" V 8925 2450 50  0000 C CNN
 F 2 "Diodes_THT:D_DO-35_SOD27_P2.54mm_Vertical_AnodeUp" H 8975 2225 50  0001 C CNN
 F 3 "" H 8975 2225 50  0001 C CNN
@@
 U 1 1 5C6DDDFD
 P 3350 5625
-F 0 "C5" H 3375 5725 50  0000 L CNN
-F 1 "10u" H 3375 5525 50  0000 L CNN
+F 0 "C5" H 3400 5525 50  0000 L CNN
+F 1 "10u" H 3400 5725 50  0000 L CNN
 F 2 "Capacitors_THT:CP_Radial_D4.0mm_P2.00mm" H 3388 5475 50  0001 C CNN
 F 3 "" H 3350 5625 50  0001 C CNN
@@
 U 1 1 5C6DEA9E
 P 3475 5200
-F 0 "C6" H 3500 5300 50  0000 L CNN
+F 0 "C6" H 3275 5200 50  0000 L CNN
 F 1 "100u" H 3500 5100 50  0000 L CNN
 F 2 "Capacitors_THT:CP_Radial_D4.0mm_P2.00mm" H 3513 5050 50  0001 C CNN
@@
 U 1 1 5C77AFCD
 P 3700 4975
-F 0 "L1" V 3550 5000 50  0000 C CNN
-F 1 "Ferrite_Bead" V 3850 4975 50  0000 C CNN
+F 0 "L1" V 3625 4925 50  0000 C CNN
+F 1 "Ferrite_Bead" V 3750 5150 50  0000 C CNN
 F 2 "Inductors_THT:L_Axial_L6.6mm_D2.7mm_P2.54mm_Vertical_Vishay_IM-2" V 3630 4975 50  0001 C CNN
 F 3 "" H 3700 4975 50  0001 C CNN
@@
 	2600 2725 2875 2725
 $Comp
-L C C7
+L R R13
 U 1 1 5C77CB15
 P 4150 2875
-F 0 "C7" H 4025 3050 50  0000 L CNN
-F 1 "10n" H 4000 2975 50  0000 L CNN
-F 2 "Capacitors_SMD:C_0805_HandSoldering" H 4188 2725 50  0001 C CNN
+F 0 "R13" H 3950 2875 50  0000 L CNN
+F 1 "1M" H 4225 2875 50  0000 L CNN
+F 2 "Resistors_SMD:R_0805_HandSoldering" H 4188 2725 50  0001 C CNN
 F 3 "" H 4150 2875 50  0001 C CNN
 	1    4150 2875
@@
 U 1 1 5C782EE1
 P 7125 2425
-F 0 "R10" V 6950 2425 50  0000 C CNN
-F 1 "10k" V 7025 2425 50  0000 C CNN
+F 0 "R10" V 7025 2425 50  0000 C CNN
+F 1 "10k" V 7225 2425 50  0000 C CNN
 F 2 "Resistors_SMD:R_0805_HandSoldering" V 7055 2425 50  0001 C CNN
 F 3 "" H 7125 2425 50  0001 C CNN
@@
 U 1 1 5C7E5B6D
 P 6950 2625
-F 0 "R11" H 7050 2600 50  0000 C CNN
-F 1 "10k" H 7075 2675 50  0000 C CNN
+F 0 "R11" H 7075 2700 50  0000 C CNN
+F 1 "10k" H 6825 2700 50  0000 C CNN
 F 2 "Resistors_SMD:R_0805_HandSoldering" V 6880 2625 50  0001 C CNN
 F 3 "" H 6950 2625 50  0001 C CNN
@@
 	6950 2850 6950 2775
 $Comp
-L C C2
+L R R12
 U 1 1 5C7E63D8
 P 2750 2925
-F 0 "C2" H 2625 3100 50  0000 L CNN
-F 1 "1n" H 2600 3025 50  0000 L CNN
-F 2 "Capacitors_SMD:C_0805_HandSoldering" H 2788 2775 50  0001 C CNN
+F 0 "R12" H 2550 2925 50  0000 L CNN
+F 1 "1M" H 2800 2925 50  0000 L CNN
+F 2 "Resistors_SMD:R_0805_HandSoldering" H 2788 2775 50  0001 C CNN
 F 3 "" H 2750 2925 50  0001 C CNN
 	1    2750 2925
@@
 U 1 1 5C7E700C
 P 7375 1450
-F 0 "R7" V 7275 1725 50  0000 C CNN
-F 1 "100k" V 7325 1625 50  0000 C CNN
+F 0 "R7" V 7475 1450 50  0000 C CNN
+F 1 "100k" V 7375 1450 50  0000 C CNN
 F 2 "Resistors_SMD:R_0805_HandSoldering" V 7305 1450 50  0001 C CNN
 F 3 "" H 7375 1450 50  0001 C CNN
@@
 U 1 1 5C7E7C56
 P 4100 4775
-F 0 "C9" H 3975 4950 50  0000 L CNN
+F 0 "C9" H 3975 4975 50  0000 L CNN
 F 1 "100n" H 3950 4875 50  0000 L CNN
 F 2 "Capacitors_SMD:C_0805_HandSoldering" H 4138 4625 50  0001 C CNN
@@
 U 1 1 5C7EA466
 P 3800 5650
-F 0 "C3" H 3675 5825 50  0000 L CNN
-F 1 "100n" H 3650 5750 50  0000 L CNN
+F 0 "C3" H 3675 5775 50  0000 L CNN
+F 1 "100n" H 3600 5550 50  0000 L CNN
 F 2 "Capacitors_SMD:C_0805_HandSoldering" H 3838 5500 50  0001 C CNN
 F 3 "" H 3800 5650 50  0001 C CNN
@@
 U 1 1 5C7EB7B4
 P 3875 4775
-F 0 "C8" H 3900 4875 50  0000 L CNN
+F 0 "C8" H 3925 4600 50  0000 L CNN
 F 1 "10u" H 3900 4675 50  0000 L CNN
 F 2 "Capacitors_THT:CP_Radial_D6.3mm_P2.50mm" H 3875 4775 50  0001 C CNN
@@
 U 1 1 5C7EBBF2
 P 8575 5075
-F 0 "C11" H 8450 5250 50  0000 L CNN
-F 1 "100n" H 8425 5175 50  0000 L CNN
+F 0 "C11" H 8425 5250 50  0000 L CNN
+F 1 "100n" H 8375 5175 50  0000 L CNN
 F 2 "Capacitors_SMD:C_0805_HandSoldering" H 8613 4925 50  0001 C CNN
 F 3 "" H 8575 5075 50  0001 C CNN
@@
 U 1 1 5C7EBFA0
 P 9275 5075
-F 0 "C12" H 9150 5250 50  0000 L CNN
-F 1 "100n" H 9125 5175 50  0000 L CNN
+F 0 "C12" H 9100 5250 50  0000 L CNN
+F 1 "100n" H 9075 5175 50  0000 L CNN
 F 2 "Capacitors_SMD:C_0805_HandSoldering" H 9313 4925 50  0001 C CNN
 F 3 "" H 9275 5075 50  0001 C CNN
